File: machine/schematic-pi/schematic-pi.sch (KiCad schematic (older format))
At the start: 6 parts, among them J1 Raspberry Pi PLEASE SEE (http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, K1 T9AS1D12-5, Q1 2N7000, SW1 Single Pole Dual Throw Switch, SW2 SW_Reed_SPDT

Commit message: Update schematic
Parts:
- R1: value Random resistance -> Random resistance representing AC circuit
Connections:
- net at J1.1 (3V3): no longer SW1.2 (B)
- net at J1.6 (GND): now also SW1.2 (B)
Changed lines of the file:
@@
 $EndDescr
-Wire Wire Line
-	3000 1750 3000 2000
 Wire Wire Line
 	1700 2800 2100 2800
@@
 Wire Wire Line
 	1300 1350 1700 1350
-Wire Wire Line
-	900  1750 3000 1750
-Wire Wire Line
-	900  1450 900  1750
+Wire Notes Line
+	6050 6250 800  6250
+Wire Notes Line
+	800  6250 800  650
+Wire Notes Line
+	800  650  6050 650
+Wire Notes Line
+	6050 650  6050 6250
+Text Notes 1350 650  0    79   ~ 16
+On the Table: Raspberry Pi, Breadboard, Switch, N-Type MOSFET
+Wire Notes Line
+	10600 650  6350 650
+Wire Notes Line
+	6350 650  6350 2700
+Wire Notes Line
+	6350 2700 10600 2700
+Wire Notes Line
+	10600 2700 10600 650
+Text Notes 7350 650  0    79   ~ 16
+On the Floor: Power Supply, Relay
+Wire Notes Line
+	10600 3100 6350 3100
+Wire Notes Line
+	6350 3100 6350 5150
+Wire Notes Line
+	6350 5150 10600 5150
+Wire Notes Line
+	10600 5150 10600 3100
+Text Notes 7550 3100 0    79   ~ 16
+Door Area: Open Sensor, Open Sign Above Door
+Wire Wire Line
+	9100 1200 9100 3750
+Wire Wire Line
+	8950 3250 8950 3550
+Wire Wire Line
+	8450 3650 8450 5550
+$Comp
+L Device:R R1
+U 1 1 5D79CC3E
+P 8950 4600
+F 0 "R1" V 8743 4600 50  0000 C CNN
+F 1 "Random resistance representing AC circuit" V 8834 4600 50  0000 C CNN
+F 2 "" V 8880 4600 50  0001 C CNN
+F 3 "~" H 8950 4600 50  0001 C CNN
+	1    8950 4600
+	0    1    1    0
+$EndComp
+Wire Wire Line
+	10450 4600 10450 1000
+Wire Wire Line
+	9100 4600 10450 4600
+Wire Wire Line
+	8800 4600 7300 4600
+$Comp
+L Switch:SW_SPDT SW1
+U 1 1 5D7833A7
+P 1100 1450
+F 0 "SW1" H 1100 1735 50  0000 C CNN
+F 1 "Single Pole Dual Throw Switch" H 1100 1644 50  0000 L CNN
+F 2 "" H 1100 1450 50  0001 C CNN
+F 3 "~" H 1100 1450 50  0001 C CNN
+	1    1100 1450
+	1    0    0    -1
+$EndComp
+$Comp
+L Switch:SW_Reed_SPDT SW2
+U 1 1 5D7A9C3D
+P 8650 3650
+F 0 "SW2" H 8700 3931 50  0000 C CNN
+F 1 "SW_Reed_SPDT" H 8700 3840 50  0000 C CNN
+F 2 "" H 8650 3650 50  0001 C CNN
+F 3 "~" H 8650 3650 50  0001 C CNN
+	1    8650 3650
+	1    0    0    -1
+$EndComp
+$Comp
+L Relay:SANYOU_SRD_Form_C K1
+U 1 1 5D786456
+P 7100 2000
+F 0 "K1" H 7530 2046 50  0000 L CNN
+F 1 "T9AS1D12-5" H 7530 1955 50  0000 L CNN
+F 2 "Relay_THT:Relay_SPDT_SANYOU_SRD_Series_Form_C" H 7550 1950 50  0001 L CNN
+F 3 "http://www.sanyourelay.ca/public/products/pdf/SRD.pdf" H 7100 2000 50  0001 C CNN
+	1    7100 2000
+	1    0    0    -1
+$EndComp
 $Comp
 L Connector:Raspberry_Pi_2_3 J1
@@
 	1    0    0    -1
 $EndComp
-Wire Notes Line
-	6050 6250 800  6250
-Wire Notes Line
-	800  6250 800  650
-Wire Notes Line
-	800  650  6050 650
-Wire Notes Line
-	6050 650  6050 6250
-Text Notes 1350 650  0    79   ~ 16
-On the Table: Raspberry Pi, Breadboard, Switch, N-Type MOSFET
-Wire Notes Line
-	10600 650  6350 650
-Wire Notes Line
-	6350 650  6350 2700
-Wire Notes Line
-	6350 2700 10600 2700
-Wire Notes Line
-	10600 2700 10600 650
-Text Notes 7350 650  0    79   ~ 16
-On the Floor: Power Supply, Relay
-Wire Notes Line
-	10600 3100 6350 3100
-Wire Notes Line
-	6350 3100 6350 5150
-Wire Notes Line
-	6350 5150 10600 5150
-Wire Notes Line
-	10600 5150 10600 3100
-Text Notes 7550 3100 0    79   ~ 16
-Door Area: Open Sensor, Open Sign Above Door
-Wire Wire Line
-	9100 1200 9100 3750
-Wire Wire Line
-	8950 3250 8950 3550
-Wire Wire Line
-	8450 3650 8450 5550
-$Comp
-L Device:R R1
-U 1 1 5D79CC3E
-P 8950 4600
-F 0 "R1" V 8743 4600 50  0000 C CNN
-F 1 "Random resistance" V 8834 4600 50  0000 C CNN
-F 2 "" V 8880 4600 50  0001 C CNN
-F 3 "~" H 8950 4600 50  0001 C CNN
-	1    8950 4600
-	0    1    1    0
-$EndComp
-Wire Wire Line
-	10450 4600 10450 1000
-Wire Wire Line
-	9100 4600 10450 4600
-Wire Wire Line
-	8800 4600 7300 4600
-$Comp
-L Switch:SW_SPDT SW1
-U 1 1 5D7833A7
-P 1100 1450
-F 0 "SW1" H 1100 1735 50  0000 C CNN
-F 1 "Single Pole Dual Throw Switch" H 1100 1644 50  0000 L CNN
-F 2 "" H 1100 1450 50  0001 C CNN
-F 3 "~" H 1100 1450 50  0001 C CNN
-	1    1100 1450
-	1    0    0    -1
-$EndComp
-$Comp
-L Switch:SW_Reed_SPDT SW2
-U 1 1 5D7A9C3D
-P 8650 3650
-F 0 "SW2" H 8700 3931 50  0000 C CNN
-F 1 "SW_Reed_SPDT" H 8700 3840 50  0000 C CNN
-F 2 "" H 8650 3650 50  0001 C CNN
-F 3 "~" H 8650 3650 50  0001 C CNN
-	1    8650 3650
-	1    0    0    -1
-$EndComp
-$Comp
-L Relay:SANYOU_SRD_Form_C K1
-U 1 1 5D786456
-P 7100 2000
-F 0 "K1" H 7530 2046 50  0000 L CNN
-F 1 "T9AS1D12-5" H 7530 1955 50  0000 L CNN
-F 2 "Relay_THT:Relay_SPDT_SANYOU_SRD_Series_Form_C" H 7550 1950 50  0001 L CNN
-F 3 "http://www.sanyourelay.ca/public/products/pdf/SRD.pdf" H 7100 2000 50  0001 C CNN
-	1    7100 2000
-	1    0    0    -1
-$EndComp
+Wire Wire Line
+	2500 4600 900  4600
+Wire Wire Line
+	900  4600 900  1450
 $EndSCHEMATC

Commit message: Update schematic to include both transistors & both driving pins
Parts:
- added Q2: 2N7000, Package_TO_SOT_THT:TO-92_Inline, symbol Transistor_FET:2N7000
Connections:
- net at J1.15 (GPIO22), Q1.2 (G): now also J1.16 (GPIO23), Q2.2 (G)
- net at J1.39 (GND), Q1.1 (S): now also Q2.1 (S)
- net at K1.2, Q1.3 (D): now also Q2.3 (D)
Changed lines of the file:
@@
 	2100 3500 1800 3500
 Wire Wire Line
-	1800 3500 1800 5500
-Wire Wire Line
-	1800 5500 5200 5500
+	1800 3500 1800 3600
+Wire Wire Line
+	1800 5500 4700 5500
 Wire Wire Line
 	5200 5500 5200 2500
@@
 Wire Wire Line
 	900  4600 900  1450
+Wire Wire Line
+	2100 3600 1800 3600
+Connection ~ 1800 3600
+Wire Wire Line
+	1800 3600 1800 5500
+$Comp
+L Transistor_FET:2N7000 Q2
+U 1 1 5DB75C8F
+P 4900 2500
+F 0 "Q2" H 5106 2546 50  0000 L CNN
+F 1 "2N7000" H 5106 2455 50  0000 L CNN
+F 2 "Package_TO_SOT_THT:TO-92_Inline" H 5100 2425 50  0001 L CIN
+F 3 "https://www.fairchildsemi.com/datasheets/2N/2N7000.pdf" H 4900 2500 50  0001 L CNN
+	1    4900 2500
+	1    0    0    -1
+$EndComp
+Wire Wire Line
+	5500 2300 5000 2300
+Connection ~ 5500 2300
+Wire Wire Line
+	5000 2700 5500 2700
+Connection ~ 5500 2700
+Wire Wire Line
+	4700 2500 4700 5500
+Connection ~ 4700 5500
+Wire Wire Line
+	4700 5500 5200 5500
 $EndSCHEMATC
